File: Circuit/PWM Multiplexer/final version/PWM_Multiplexer.kicad_pcb (KiCad board)
At the start: 2 copper layers, 80.3 x 79.2 mm, 71 parts, among them J1 JST connector, Q1 S8050, Q10 S8050, Q11 S8050, Q12 S8050, Q13 S8050, Q14 S8050, Q2 S8050, Q3 S8050, Q4 S8050, Q5 S8050, Q6 S8050, Q7 S8050, Q8 S8050, Q9 S8050, U1 PC817, U2 PC817, U3 PC817, U4 PC817, U5 L7805, U6 74HC137, U7 74HC137

Commit message: added .step file and some media
Routing:
- net +12V: track 86.4 -> 144.6 mm
- net GND: track 601.6 -> 658.4 mm
Changed lines of the file:
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@@
   (segment (start 112.268 117.2972) (end 112.268 122.2631) (width 1.5) (layer "F.Cu") (net 1))
   (segment (start 158.540153 63.726753) (end 157.5914 62.778) (width 1.5) (layer "B.Cu") (net 1))
+  (segment (start 116.5272 122.202) (end 117.994962 122.202) (width 1.5) (layer "B.Cu") (net 1))
   (segment (start 158.540153 71.877847) (end 158.540153 82.901447) (width 1.5) (layer "B.Cu") (net 1))
   (segment (start 156.6164 117.729381) (end 156.6164 117.896) (width 1.5) (layer "B.Cu") (net 1))
+  (segment (start 157.211019 124.968) (end 158.540153 123.638866) (width 1.5) (layer "B.Cu") (net 1))
   (segment (start 158.540153 93.925047) (end 156.6164 95.8488) (width 1.5) (layer "B.Cu") (net 1))
+  (segment (start 158.540153 123.638866) (end 158.540153 115.805628) (width 1.5) (layer "B.Cu") (net 1))
   (segment (start 158.540153 82.901447) (end 156.6164 84.8252) (width 1.5) (layer "B.Cu") (net 1))
   (segment (start 158.540153 82.901447) (end 158.540153 93.925047) (width 1.5) (layer "B.Cu") (net 1))
+  (segment (start 120.760962 124.968) (end 157.211019 124.968) (width 1.5) (layer "B.Cu") (net 1))
+  (segment (start 116.5272 122.202) (end 116.5272 121.5564) (width 1.5) (layer "B.Cu") (net 1))
   (segment (start 157.5914 62.778) (end 156.6164 62.778) (width 1.5) (layer "B.Cu") (net 1))
   (segment (start 158.540153 115.805628) (end 156.6164 117.729381) (width 1.5) (layer "B.Cu") (net 1))
   (segment (start 158.540153 71.877847) (end 156.6164 73.8016) (width 1.5) (layer "B.Cu") (net 1))
   (segment (start 158.540153 104.948647) (end 158.540153 115.805628) (width 1.5) (layer "B.Cu") (net 1))
+  (segment (start 117.994962 122.202) (end 120.760962 124.968) (width 1.5) (layer "B.Cu") (net 1))
   (segment (start 158.540153 93.925047) (end 158.540153 104.948647) (width 1.5) (layer "B.Cu") (net 1))
   (segment (start 158.540153 71.877847) (end 158.540153 63.726753) (width 1.5) (layer "B.Cu") (net 1))
+  (segment (start 116.5272 121.5564) (end 112.268 117.2972) (width 1.5) (layer "B.Cu") (net 1))
   (segment (start 158.540153 104.948647) (end 156.6164 106.8724) (width 1.5) (layer "B.Cu") (net 1))
   (segment (start 164.2072 125.903729) (end 164.2364 125.932929) (width 0.8) (layer "F.Cu") (net 2))
@@
   (segment (start 144.9 108.240814) (end 144.9 103.465614) (width 0.8) (layer "F.Cu") (net 2))
   (segment (start 144.9 108.240814) (end 144.072786 107.4136) (width 0.8) (layer "F.Cu") (net 2))
+  (segment (start 109.728 116.541196) (end 109.728 117.2972) (width 1.5) (layer "B.Cu") (net 2))
+  (segment (start 135.988162 101.0132) (end 127.47 109.531362) (width 1.5) (layer "B.Cu") (net 2))
+  (segment (start 149.5044 95.220638) (end 146.558 98.167038) (width 1.5) (layer "B.Cu") (net 2))
+  (segment (start 146.558 98.167038) (end 146.558 98.672962) (width 1.5) (layer "B.Cu") (net 2))
+  (segment (start 127.47 114.306562) (end 125.872866 115.903696) (width 1.5) (layer "B.Cu") (net 2))
+  (segment (start 114.1705 115.903696) (end 113.614004 115.3472) (width 1.5) (layer "B.Cu") (net 2))
+  (segment (start 110.921996 115.3472) (end 109.728 116.541196) (width 1.5) (layer "B.Cu") (net 2))
   (segment (start 149.5044 61.595) (end 149.5044 91.313) (width 1.5) (layer "B.Cu") (net 2))
+  (segment (start 149.5044 91.313) (end 149.5044 95.220638) (width 1.5) (layer "B.Cu") (net 2))
+  (segment (start 144.217762 101.0132) (end 135.988162 101.0132) (width 1.5) (layer "B.Cu") (net 2))
+  (segment (start 127.47 109.531362) (end 127.47 114.306562) (width 1.5) (layer "B.Cu") (net 2))
+  (segment (start 113.614004 115.3472) (end 110.921996 115.3472) (width 1.5) (layer "B.Cu") (net 2))
+  (segment (start 125.872866 115.903696) (end 114.1705 115.903696) (width 1.5) (layer "B.Cu") (net 2))
+  (segment (start 146.558 98.672962) (end 144.217762 101.0132) (width 1.5) (layer "B.Cu") (net 2))
   (segment (start 91.8348 105.0406) (end 91.8348 120.5764) (width 0.8) (layer "F.Cu") (net 3))
   (segment (start 91.8348 120.5764) (end 91.5708 120.8404) (width 0.8) (layer "F.Cu") (net 3))
